File: hw/SemiSemafor/SemiSemafor.kicad_sch (KiCad schematic)
At the start: 40 parts, among them J1 USB_PCB, J2 ESP-Programing_conector, SW1 SW_DIP_x01, SW2 SW_DIP_x01, U1 LD39200, U2 ESP32-C3-MINI-1

Commit message: V2.0 (Circuit)
Parts:
- renumbered D6 to D11, D11 to D6
Connections:
- net at D10.1 (DOUT): now also D11.3 (DIN); no longer D12.3 (DIN)
- net at D11.1 (DOUT): now also D12.3 (DIN); no longer D7.3 (DIN)
- net at D6.1 (DOUT): now also D7.3 (DIN); no longer D11.3 (DIN)
Other:
- moved on the sheet: D10, D11, D7, D8, D9
Changed lines of the file:
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@@
     )
   )
-  (symbol (lib_name "WS2812B_1") (lib_id "LED:WS2812B") (at 91.44 147.32 0) (unit 1)
-    (in_bom yes) (on_board yes) (dnp no)
-    (property "Reference" "D8" (at 99.06 143.51 0)
-      (effects (font (size 1.27 1.27)))
-    )
-    (property "Value" "WS2812B" (at 96.52 140.97 0)
-      (effects (font (size 1.27 1.27)))
-    )
-    (property "Footprint" "LED_SMD:LED_WS2812B-2020_PLCC4_2.0x2.0mm" (at 92.71 154.94 0)
-      (effects (font (size 1.27 1.27)) (justify left top) hide)
-    )
-    (property "Datasheet" "https://cdn-shop.adafruit.com/datasheets/WS2812B.pdf" (at 92.71 156.845 0)
-      (effects (font (size 1.27 1.27)) (justify left top) hide)
-    )
-    (property "LCSC" "C965555" (at 97.155 160.02 0)
-      (effects (font (size 1.27 1.27)) hide)
-    )
-    (property "JLCPCB_CORRECTION" "" (at 96.52 161.925 0)
+  (symbol (lib_name "WS2812B_1") (lib_id "LED:WS2812B") (at 68.58 147.32 0) (unit 1)
+    (in_bom yes) (on_board yes) (dnp no)
+    (property "Reference" "D8" (at 76.2 143.51 0)
+      (effects (font (size 1.27 1.27)))
+    )
+    (property "Value" "WS2812B" (at 73.66 140.97 0)
+      (effects (font (size 1.27 1.27)))
+    )
+    (property "Footprint" "LED_SMD:LED_WS2812B-2020_PLCC4_2.0x2.0mm" (at 69.85 154.94 0)
+      (effects (font (size 1.27 1.27)) (justify left top) hide)
+    )
+    (property "Datasheet" "https://cdn-shop.adafruit.com/datasheets/WS2812B.pdf" (at 69.85 156.845 0)
+      (effects (font (size 1.27 1.27)) (justify left top) hide)
+    )
+    (property "LCSC" "C965555" (at 74.295 160.02 0)
+      (effects (font (size 1.27 1.27)) hide)
+    )
+    (property "JLCPCB_CORRECTION" "" (at 73.66 161.925 0)
       (effects (font (size 1.27 1.27)) hide)
     )
@@
     )
   )
-  (symbol (lib_name "WS2812B_1") (lib_id "LED:WS2812B") (at 114.3 147.32 0) (unit 1)
-    (in_bom yes) (on_board yes) (dnp no)
-    (property "Reference" "D9" (at 121.92 143.51 0)
-      (effects (font (size 1.27 1.27)))
-    )
-    (property "Value" "WS2812B" (at 119.38 140.97 0)
-      (effects (font (size 1.27 1.27)))
-    )
-    (property "Footprint" "LED_SMD:LED_WS2812B-2020_PLCC4_2.0x2.0mm" (at 115.57 154.94 0)
-      (effects (font (size 1.27 1.27)) (justify left top) hide)
-    )
-    (property "Datasheet" "https://cdn-shop.adafruit.com/datasheets/WS2812B.pdf" (at 115.57 156.845 0)
-      (effects (font (size 1.27 1.27)) (justify left top) hide)
-    )
-    (property "LCSC" "C965555" (at 120.015 160.02 0)
-      (effects (font (size 1.27 1.27)) hide)
-    )
-    (property "JLCPCB_CORRECTION" "" (at 119.38 161.925 0)
+  (symbol (lib_name "WS2812B_1") (lib_id "LED:WS2812B") (at 91.44 147.32 0) (unit 1)
+    (in_bom yes) (on_board yes) (dnp no)
+    (property "Reference" "D9" (at 99.06 143.51 0)
+      (effects (font (size 1.27 1.27)))
+    )
+    (property "Value" "WS2812B" (at 96.52 140.97 0)
+      (effects (font (size 1.27 1.27)))
+    )
+    (property "Footprint" "LED_SMD:LED_WS2812B-2020_PLCC4_2.0x2.0mm" (at 92.71 154.94 0)
+      (effects (font (size 1.27 1.27)) (justify left top) hide)
+    )
+    (property "Datasheet" "https://cdn-shop.adafruit.com/datasheets/WS2812B.pdf" (at 92.71 156.845 0)
+      (effects (font (size 1.27 1.27)) (justify left top) hide)
+    )
+    (property "LCSC" "C965555" (at 97.155 160.02 0)
+      (effects (font (size 1.27 1.27)) hide)
+    )
+    (property "JLCPCB_CORRECTION" "" (at 96.52 161.925 0)
       (effects (font (size 1.27 1.27)) hide)
     )
@@
     )
   )
-  (symbol (lib_name "WS2812B_1") (lib_id "LED:WS2812B") (at 137.16 147.32 0) (unit 1)
-    (in_bom yes) (on_board yes) (dnp no)
-    (property "Reference" "D10" (at 144.78 143.51 0)
-      (effects (font (size 1.27 1.27)))
-    )
-    (property "Value" "WS2812B" (at 142.24 140.97 0)
-      (effects (font (size 1.27 1.27)))
-    )
-    (property "Footprint" "LED_SMD:LED_WS2812B-2020_PLCC4_2.0x2.0mm" (at 138.43 154.94 0)
-      (effects (font (size 1.27 1.27)) (justify left top) hide)
-    )
-    (property "Datasheet" "https://cdn-shop.adafruit.com/datasheets/WS2812B.pdf" (at 138.43 156.845 0)
-      (effects (font (size 1.27 1.27)) (justify left top) hide)
-    )
-    (property "LCSC" "C965555" (at 142.875 160.02 0)
-      (effects (font (size 1.27 1.27)) hide)
-    )
-    (property "JLCPCB_CORRECTION" "" (at 142.24 161.925 0)
+  (symbol (lib_name "WS2812B_1") (lib_id "LED:WS2812B") (at 114.3 147.32 0) (unit 1)
+    (in_bom yes) (on_board yes) (dnp no)
+    (property "Reference" "D10" (at 121.92 143.51 0)
+      (effects (font (size 1.27 1.27)))
+    )
+    (property "Value" "WS2812B" (at 119.38 140.97 0)
+      (effects (font (size 1.27 1.27)))
+    )
+    (property "Footprint" "LED_SMD:LED_WS2812B-2020_PLCC4_2.0x2.0mm" (at 115.57 154.94 0)
+      (effects (font (size 1.27 1.27)) (justify left top) hide)
+    )
+    (property "Datasheet" "https://cdn-shop.adafruit.com/datasheets/WS2812B.pdf" (at 115.57 156.845 0)
+      (effects (font (size 1.27 1.27)) (justify left top) hide)
+    )
+    (property "LCSC" "C965555" (at 120.015 160.02 0)
+      (effects (font (size 1.27 1.27)) hide)
+    )
+    (property "JLCPCB_CORRECTION" "" (at 119.38 161.925 0)
       (effects (font (size 1.27 1.27)) hide)
     )
@@
     )
   )
-  (symbol (lib_name "WS2812B_1") (lib_id "LED:WS2812B") (at 45.72 147.32 0) (unit 1)
-    (in_bom yes) (on_board yes) (dnp no)
-    (property "Reference" "D6" (at 53.34 143.51 0)
-      (effects (font (size 1.27 1.27)))
-    )
-    (property "Value" "WS2812B" (at 50.8 140.97 0)
-      (effects (font (size 1.27 1.27)))
-    )
-    (property "Footprint" "LED_SMD:LED_WS2812B-2020_PLCC4_2.0x2.0mm" (at 46.99 154.94 0)
-      (effects (font (size 1.27 1.27)) (justify left top) hide)
-    )
-    (property "Datasheet" "https://cdn-shop.adafruit.com/datasheets/WS2812B.pdf" (at 46.99 156.845 0)
-      (effects (font (size 1.27 1.27)) (justify left top) hide)
-    )
-    (property "LCSC" "C965555" (at 51.435 160.02 0)
-      (effects (font (size 1.27 1.27)) hide)
-    )
-    (property "JLCPCB_CORRECTION" "" (at 50.8 161.925 0)
+  (symbol (lib_name "WS2812B_1") (lib_id "LED:WS2812B") (at 137.16 147.32 0) (unit 1)
+    (in_bom yes) (on_board yes) (dnp no)
+    (property "Reference" "D11" (at 144.78 143.51 0)
+      (effects (font (size 1.27 1.27)))
+    )
+    (property "Value" "WS2812B" (at 142.24 140.97 0)
+      (effects (font (size 1.27 1.27)))
+    )
+    (property "Footprint" "LED_SMD:LED_WS2812B-2020_PLCC4_2.0x2.0mm" (at 138.43 154.94 0)
+      (effects (font (size 1.27 1.27)) (justify left top) hide)
+    )
+    (property "Datasheet" "https://cdn-shop.adafruit.com/datasheets/WS2812B.pdf" (at 138.43 156.845 0)
+      (effects (font (size 1.27 1.27)) (justify left top) hide)
+    )
+    (property "LCSC" "C965555" (at 142.875 160.02 0)
+      (effects (font (size 1.27 1.27)) hide)
+    )
+    (property "JLCPCB_CORRECTION" "" (at 142.24 161.925 0)
       (effects (font (size 1.27 1.27)) hide)
     )
@@
       (project "SemiSemafor"
         (path "/fb82d987-26cf-425e-8e99-22ecb59c8a96"
-          (reference "D6") (unit 1)
+          (reference "D11") (unit 1)
         )
       )
@@
     )
   )
-  (symbol (lib_name "WS2812B_1") (lib_id "LED:WS2812B") (at 68.58 147.32 0) (unit 1)
-    (in_bom yes) (on_board yes) (dnp no)
-    (property "Reference" "D7" (at 76.2 143.51 0)
-      (effects (font (size 1.27 1.27)))
-    )
-    (property "Value" "WS2812B" (at 73.66 140.97 0)
-      (effects (font (size 1.27 1.27)))
-    )
-    (property "Footprint" "LED_SMD:LED_WS2812B-2020_PLCC4_2.0x2.0mm" (at 69.85 154.94 0)
-      (effects (font (size 1.27 1.27)) (justify left top) hide)
-    )
-    (property "Datasheet" "https://cdn-shop.adafruit.com/datasheets/WS2812B.pdf" (at 69.85 156.845 0)
-      (effects (font (size 1.27 1.27)) (justify left top) hide)
-    )
-    (property "LCSC" "C965555" (at 74.295 160.02 0)
-      (effects (font (size 1.27 1.27)) hide)
-    )
-    (property "JLCPCB_CORRECTION" "" (at 73.66 161.925 0)
+  (symbol (lib_name "WS2812B_1") (lib_id "LED:WS2812B") (at 45.72 147.32 0) (unit 1)
+    (in_bom yes) (on_board yes) (dnp no)
+    (property "Reference" "D7" (at 53.34 143.51 0)
+      (effects (font (size 1.27 1.27)))
+    )
+    (property "Value" "WS2812B" (at 50.8 140.97 0)
+      (effects (font (size 1.27 1.27)))
+    )
+    (property "Footprint" "LED_SMD:LED_WS2812B-2020_PLCC4_2.0x2.0mm" (at 46.99 154.94 0)
+      (effects (font (size 1.27 1.27)) (justify left top) hide)
+    )
+    (property "Datasheet" "https://cdn-shop.adafruit.com/datasheets/WS2812B.pdf" (at 46.99 156.845 0)
+      (effects (font (size 1.27 1.27)) (justify left top) hide)
+    )
+    (property "LCSC" "C965555" (at 51.435 160.02 0)
+      (effects (font (size 1.27 1.27)) hide)
+    )
+    (property "JLCPCB_CORRECTION" "" (at 50.8 161.925 0)
       (effects (font (size 1.27 1.27)) hide)
     )
@@
   (symbol (lib_name "WS2812B_1") (lib_id "LED:WS2812B") (at 160.02 114.3 0) (unit 1)
     (in_bom yes) (on_board yes) (dnp no)
-    (property "Reference" "D11" (at 167.64 110.49 0)
+    (property "Reference" "D6" (at 167.64 110.49 0)
       (effects (font (size 1.27 1.27)))
     )
@@
       (project "SemiSemafor"
         (path "/fb82d987-26cf-425e-8e99-22ecb59c8a96"
-          (reference "D11") (unit 1)
-        )
-      )
+          (reference "D6") (unit 1)
+        )
+      )

Commit message: Small ring
Parts:
- C1, C10, C11, C12, C13, C14, C15, C2, C3, C4, C5, C9: footprint Capacitor_SMD:C_0402_1005Metric -> Capacitor_SMD:C_0603_1608Metric; LCSC C52923 -> C14663
Changed lines of the file:
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@@
       (effects (font (size 1.27 1.27)) (justify left))
     )
-    (property "Footprint" "Capacitor_SMD:C_0402_1005Metric" (at 149.5552 151.13 0)
+    (property "Footprint" "Capacitor_SMD:C_0603_1608Metric" (at 149.5552 151.13 0)
       (effects (font (size 1.27 1.27)) hide)
     )
@@
       (effects (font (size 1.27 1.27)) hide)
     )
-    (property "LCSC" "C52923" (at 148.59 147.32 0)
+    (property "LCSC" "C14663" (at 148.59 147.32 0)
       (effects (font (size 1.27 1.27)) hide)
     )
@@
         (path "/fb82d987-26cf-425e-8e99-22ecb59c8a96"
           (reference "C13") (unit 1)
-        )
-      )
-    )
-  )
-  (symbol (lib_id "Device:C") (at 247.65 119.38 0) (unit 1)
-    (in_bom yes) (on_board yes) (dnp no) (fields_autoplaced)
-    (property "Reference" "C7" (at 251.46 118.1099 0)
-      (effects (font (size 1.27 1.27)) (justify left))
-    )
-    (property "Value" "1u" (at 251.46 120.6499 0)
-      (effects (font (size 1.27 1.27)) (justify left))
-    )
-    (property "Footprint" "Capacitor_SMD:C_0402_1005Metric" (at 248.6152 123.19 0)
-      (effects (font (size 1.27 1.27)) hide)
-    )
-    (property "Datasheet" "~" (at 247.65 119.38 0)
-      (effects (font (size 1.27 1.27)) hide)
-    )
-    (property "LCSC" "C52923" (at 247.65 119.38 0)
-      (effects (font (size 1.27 1.27)) hide)
-    )
-    (pin "1")
-    (pin "2")
-    (instances
-      (project "SemiSemafor"
-        (path "/fb82d987-26cf-425e-8e99-22ecb59c8a96"
-          (reference "C7") (unit 1)
         )
       )
@@
       (effects (font (size 1.27 1.27)) (justify left))
     )
-    (property "Footprint" "Capacitor_SMD:C_0402_1005Metric" (at 126.6952 118.11 0)
+    (property "Footprint" "Capacitor_SMD:C_0603_1608Metric" (at 126.6952 118.11 0)
       (effects (font (size 1.27 1.27)) hide)
     )
@@
       (effects (font (size 1.27 1.27)) hide)
     )
-    (property "LCSC" "C52923" (at 125.73 114.3 0)
+    (property "LCSC" "C14663" (at 125.73 114.3 0)
       (effects (font (size 1.27 1.27)) hide)
     )
@@
         (path "/fb82d987-26cf-425e-8e99-22ecb59c8a96"
           (reference "#PWR0128") (unit 1)
+        )
+      )
+    )
+  )
+  (symbol (lib_id "Device:C") (at 247.65 119.38 0) (unit 1)
+    (in_bom yes) (on_board yes) (dnp no) (fields_autoplaced)
+    (property "Reference" "C7" (at 251.46 118.1099 0)
+      (effects (font (size 1.27 1.27)) (justify left))
+    )
+    (property "Value" "1u" (at 251.46 120.6499 0)
+      (effects (font (size 1.27 1.27)) (justify left))
+    )
+    (property "Footprint" "Capacitor_SMD:C_0402_1005Metric" (at 248.6152 123.19 0)
+      (effects (font (size 1.27 1.27)) hide)
+    )
+    (property "Datasheet" "~" (at 247.65 119.38 0)
+      (effects (font (size 1.27 1.27)) hide)
+    )
+    (property "LCSC" "C52923" (at 247.65 119.38 0)
+      (effects (font (size 1.27 1.27)) hide)
+    )
+    (pin "1")
+    (pin "2")
+    (instances
+      (project "SemiSemafor"
+        (path "/fb82d987-26cf-425e-8e99-22ecb59c8a96"
+          (reference "C7") (unit 1)
         )
       )
@@
       (effects (font (size 1.27 1.27)) (justify left))
     )
-    (property "Footprint" "Capacitor_SMD:C_0402_1005Metric" (at 126.6952 151.13 0)
+    (property "Footprint" "Capacitor_SMD:C_0603_1608Metric" (at 126.6952 151.13 0)
       (effects (font (size 1.27 1.27)) hide)
     )
@@
       (effects (font (size 1.27 1.27)) hide)
     )
-    (property "LCSC" "C52923" (at 125.73 147.32 0)
+    (property "LCSC" "C14663" (at 125.73 147.32 0)
       (effects (font (size 1.27 1.27)) hide)
     )
@@
       (effects (font (size 1.27 1.27)) (justify left))
     )
-    (property "Footprint" "Capacitor_SMD:C_0402_1005Metric" (at 172.4152 118.11 0)
+    (property "Footprint" "Capacitor_SMD:C_0603_1608Metric" (at 172.4152 118.11 0)
       (effects (font (size 1.27 1.27)) hide)
     )
@@
       (effects (font (size 1.27 1.27)) hide)
     )
-    (property "LCSC" "C52923" (at 171.45 114.3 0)
+    (property "LCSC" "C14663" (at 171.45 114.3 0)
       (effects (font (size 1.27 1.27)) hide)
     )
@@
       (effects (font (size 1.27 1.27)) (justify left))
     )
-    (property "Footprint" "Capacitor_SMD:C_0402_1005Metric" (at 58.1152 118.11 0)
+    (property "Footprint" "Capacitor_SMD:C_0603_1608Metric" (at 58.1152 118.11 0)
       (effects (font (size 1.27 1.27)) hide)
     )
@@
       (effects (font (size 1.27 1.27)) hide)
     )
-    (property "LCSC" "C52923" (at 57.15 114.3 0)
+    (property "LCSC" "C14663" (at 57.15 114.3 0)
       (effects (font (size 1.27 1.27)) hide)
     )
@@
       (effects (font (size 1.27 1.27)) (justify left))
     )
-    (property "Footprint" "Capacitor_SMD:C_0402_1005Metric" (at 172.4152 151.13 0)
+    (property "Footprint" "Capacitor_SMD:C_0603_1608Metric" (at 172.4152 151.13 0)
       (effects (font (size 1.27 1.27)) hide)
     )
@@
       (effects (font (size 1.27 1.27)) hide)
     )
-    (property "LCSC" "C52923" (at 171.45 147.32 0)
+    (property "LCSC" "C14663" (at 171.45 147.32 0)
       (effects (font (size 1.27 1.27)) hide)
     )
@@
       (effects (font (size 1.27 1.27)) (justify left))
     )
-    (property "Footprint" "Capacitor_SMD:C_0402_1005Metric" (at 58.1152 151.13 0)
+    (property "Footprint" "Capacitor_SMD:C_0603_1608Metric" (at 58.1152 151.13 0)
       (effects (font (size 1.27 1.27)) hide)
     )
@@
       (effects (font (size 1.27 1.27)) hide)
     )
-    (property "LCSC" "C52923" (at 57.15 147.32 0)
+    (property "LCSC" "C14663" (at 57.15 147.32 0)
       (effects (font (size 1.27 1.27)) hide)
     )
@@
       (effects (font (size 1.27 1.27)) (justify left))
     )
-    (property "Footprint" "Capacitor_SMD:C_0402_1005Metric" (at 80.9752 151.13 0)
+    (property "Footprint" "Capacitor_SMD:C_0603_1608Metric" (at 80.9752 151.13 0)
       (effects (font (size 1.27 1.27)) hide)
     )
@@
       (effects (font (size 1.27 1.27)) hide)
     )
-    (property "LCSC" "C52923" (at 80.01 147.32 0)
+    (property "LCSC" "C14663" (at 80.01 147.32 0)
       (effects (font (size 1.27 1.27)) hide)
     )
@@
       (effects (font (size 1.27 1.27)) (justify left))
     )
-    (property "Footprint" "Capacitor_SMD:C_0402_1005Metric" (at 80.9752 118.11 0)
+    (property "Footprint" "Capacitor_SMD:C_0603_1608Metric" (at 80.9752 118.11 0)
       (effects (font (size 1.27 1.27)) hide)
     )
@@
       (effects (font (size 1.27 1.27)) hide)
     )
-    (property "LCSC" "C52923" (at 80.01 114.3 0)
+    (property "LCSC" "C14663" (at 80.01 114.3 0)
       (effects (font (size 1.27 1.27)) hide)
     )
@@
       (effects (font (size 1.27 1.27)) (justify left))
     )
-    (property "Footprint" "Capacitor_SMD:C_0402_1005Metric" (at 103.8352 118.11 0)
+    (property "Footprint" "Capacitor_SMD:C_0603_1608Metric" (at 103.8352 118.11 0)
       (effects (font (size 1.27 1.27)) hide)
     )
@@
       (effects (font (size 1.27 1.27)) hide)
     )
-    (property "LCSC" "C52923" (at 102.87 114.3 0)
+    (property "LCSC" "C14663" (at 102.87 114.3 0)
       (effects (font (size 1.27 1.27)) hide)
     )
@@
       (effects (font (size 1.27 1.27)) (justify left))
     )
-    (property "Footprint" "Capacitor_SMD:C_0402_1005Metric" (at 149.5552 118.11 0)
+    (property "Footprint" "Capacitor_SMD:C_0603_1608Metric" (at 149.5552 118.11 0)
       (effects (font (size 1.27 1.27)) hide)
     )
@@
       (effects (font (size 1.27 1.27)) hide)
     )
-    (property "LCSC" "C52923" (at 148.59 114.3 0)
+    (property "LCSC" "C14663" (at 148.59 114.3 0)
       (effects (font (size 1.27 1.27)) hide)
     )
@@
       (effects (font (size 1.27 1.27)) (justify left))
     )
-    (property "Footprint" "Capacitor_SMD:C_0402_1005Metric" (at 103.8352 151.13 0)
+    (property "Footprint" "Capacitor_SMD:C_0603_1608Metric" (at 103.8352 151.13 0)
       (effects (font (size 1.27 1.27)) hide)
     )
@@
       (effects (font (size 1.27 1.27)) hide)
     )
-    (property "LCSC" "C52923" (at 102.87 147.32 0)
-      (effects (font (size 1.27 1.27)) hide)
-    )
+    (property "LCSC" "C14663" (at 102.87 147.32 0)
+      (effects (font (size 1.27 1.27)) hide)
+    )
