File: hw/SemiSemafor/SemiSemafor.kicad_sch (KiCad schematic)
At the start: 44 parts, among them J1 USB_PCB, J2 ESP-Programing_conector, SW1 SW_DIP_x01, SW2 SW_DIP_x01, U1 LD39200, U2 ESP32-C3-MINI-1, U3 LIS2DH12

Commit message: Correction
Parts:
- U2: JLCPCB_CORRECTION (none) -> 0;0;180
Changed lines of the file:
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@@
       (effects (font (size 1.27 1.27)) hide)
     )
-    (property "JLCPCB_CORRECTION" "" (at 156.21 46.99 0)
+    (property "JLCPCB_CORRECTION" "0;0;180" (at 156.21 46.99 0)
       (effects (font (size 1.27 1.27)) hide)
     )

Commit message: v2.1.0
Parts:
- added J3: Conn_01x02, RKL-ESP:ESP-Small-programming connector, symbol Connector_Generic:Conn_01x02
Connections:
- net BOOT: now also J3.2 (Pin_2)
- net EN: now also J3.1 (Pin_1)
Other:
- moved on the sheet: J2, R2, R3, R4, R5

Commit message: Change package of FB1
Parts:
- FB1: footprint Inductor_SMD:L_0201_0603Metric -> Inductor_SMD:L_0402_1005Metric; LCSC C160965 -> C275411
Changed lines of the file:
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@@
       (effects (font (size 1.27 1.27)))
     )
-    (property "Footprint" "Inductor_SMD:L_0201_0603Metric" (at 27.94 146.558 90)
+    (property "Footprint" "Inductor_SMD:L_0402_1005Metric" (at 27.94 146.558 90)
       (effects (font (size 1.27 1.27)) hide)
     )
@@
       (effects (font (size 1.27 1.27)) hide)
     )
-    (property "LCSC" "C160965" (at 27.94 144.78 90)
+    (property "LCSC" "C275411" (at 27.94 144.78 90)
       (effects (font (size 1.27 1.27)) hide)
     )
