File: hw/SemiSemafor/SemiSemafor.kicad_pcb (KiCad board)
At the start: 2 copper layers, 40.2 x 66.1 mm, 46 parts, among them J1 USB_PCB, J2 ESP-Programing_conector, J3 Conn_01x02, SW1 SW_DIP_x01, SW2 SW_DIP_x01, U1 LD39200, U2 ESP32-C3-MINI-1, U3 LIS2DH12

Commit message: Makefile
Parts:
- added REF**: Tab, kikit:Tab, F.Cu at (150.0, 59.6)
- added REF**: Tab, kikit:Tab, F.Cu at (139.7, 104.0)
- added REF**: Tab, kikit:Tab, F.Cu at (160.2, 104.0)
- added REF**: Tab, kikit:Tab, F.Cu at (150.0, 126.2)
Connections:
- U2 pad 7: (no net) -> +3.3V
Routing:
- net GND: vias 22 -> 24
Other:
- outline, holes or cut-outs redrawn
Changed lines of the file:
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@@
     )
   )
+  (footprint "kikit:Tab" (layer "F.Cu")
+    (at 150 59.6 -90)
+    (descr "A symbol representing annotation for tab placement")
+    (attr exclude_from_pos_files exclude_from_bom)
+    (fp_text reference "REF**" (at 0 -2 90) (layer "F.SilkS") hide
+        (effects (font (size 1 1) (thickness 0.15)))
+    )
+    (fp_text value "Tab" (at -3 -1 90) (layer "Dwgs.User")
+        (effects (font (size 1.2 1.2) (thickness 0.2)))
+    )
+    (fp_text user "KIKIT: width: 3mm" (at -5.5 0) (layer "Dwgs.User")
+        (effects (font (size 1 1) (thickness 0.15)))
+    )
+    (fp_line (start 0.25 0) (end -2.75 0)
+      (stroke (width 0.3) (type solid)) (layer "Dwgs.User"))
+    (fp_line (start 0.25 0) (end -0.75 -1)
+      (stroke (width 0.3) (type solid)) (layer "Dwgs.User"))
+    (fp_line (start 0.25 0) (end -0.75 1)
+      (stroke (width 0.3) (type solid)) (layer "Dwgs.User"))
+    (fp_line (start 0.25 1) (end 0.25 -1)
+      (stroke (width 0.3) (type solid)) (layer "Dwgs.User"))
+  )
+  (footprint "kikit:Tab" (layer "F.Cu")
+    (at 139.7 104)
+    (descr "A symbol representing annotation for tab placement")
+    (attr exclude_from_pos_files exclude_from_bom)
+    (fp_text reference "REF**" (at 0 -2) (layer "F.SilkS") hide
+        (effects (font (size 1 1) (thickness 0.15)))
+    )
+    (fp_text value "Tab" (at -3 -1) (layer "Dwgs.User")
+        (effects (font (size 1.2 1.2) (thickness 0.2)))
+    )
+    (fp_text user "KIKIT: width: 3mm" (at -5.5 0 90) (layer "Dwgs.User")
+        (effects (font (size 1 1) (thickness 0.15)))
+    )
+    (fp_line (start 0.25 0) (end -2.75 0)
+      (stroke (width 0.3) (type solid)) (layer "Dwgs.User"))
+    (fp_line (start 0.25 0) (end -0.75 -1)
+      (stroke (width 0.3) (type solid)) (layer "Dwgs.User"))
+    (fp_line (start 0.25 0) (end -0.75 1)
+      (stroke (width 0.3) (type solid)) (layer "Dwgs.User"))
+    (fp_line (start 0.25 1) (end 0.25 -1)
+      (stroke (width 0.3) (type solid)) (layer "Dwgs.User"))
+  )
   (footprint "Capacitor_SMD:C_0402_1005Metric" (layer "F.Cu")
     (at 147.91 105.97 180)
@@
     )
   )
+  (footprint "kikit:Tab" (layer "F.Cu")
+    (at 160.25 104 180)
+    (descr "A symbol representing annotation for tab placement")
+    (attr exclude_from_pos_files exclude_from_bom)
+    (fp_text reference "REF**" (at 0 -2) (layer "F.SilkS") hide
+        (effects (font (size 1 1) (thickness 0.15)))
+    )
+    (fp_text value "Tab" (at -3 -1) (layer "Dwgs.User")
+        (effects (font (size 1.2 1.2) (thickness 0.2)))
+    )
+    (fp_text user "KIKIT: width: 3mm" (at -5.5 0 90) (layer "Dwgs.User")
+        (effects (font (size 1 1) (thickness 0.15)))
+    )
+    (fp_line (start 0.25 0) (end -2.75 0)
+      (stroke (width 0.3) (type solid)) (layer "Dwgs.User"))
+    (fp_line (start 0.25 0) (end -0.75 -1)
+      (stroke (width 0.3) (type solid)) (layer "Dwgs.User"))
+    (fp_line (start 0.25 0) (end -0.75 1)
+      (stroke (width 0.3) (type solid)) (layer "Dwgs.User"))
+    (fp_line (start 0.25 1) (end 0.25 -1)
+      (stroke (width 0.3) (type solid)) (layer "Dwgs.User"))
+  )
   (footprint "LED_SMD:LED_WS2812B_PLCC4_5.0x5.0mm_P3.2mm" (layer "F.Cu")
     (at 135.883786 88.15 -60)
@@
     )
   )
+  (footprint "kikit:Tab" (layer "F.Cu")
+    (at 150 126.2 90)
+    (descr "A symbol representing annotation for tab placement")
+    (attr exclude_from_pos_files exclude_from_bom)
+    (fp_text reference "REF**" (at 0 -2 90) (layer "F.SilkS") hide
+        (effects (font (size 1 1) (thickness 0.15)))
+    )
+    (fp_text value "Tab" (at -3 -1 90) (layer "Dwgs.User")
+        (effects (font (size 1.2 1.2) (thickness 0.2)))
+    )
+    (fp_text user "KIKIT: width: 3mm" (at -5.5 0) (layer "Dwgs.User")
+        (effects (font (size 1 1) (thickness 0.15)))
+    )
+    (fp_line (start 0.25 0) (end -2.75 0)
+      (stroke (width 0.3) (type solid)) (layer "Dwgs.User"))
+    (fp_line (start 0.25 0) (end -0.75 -1)
+      (stroke (width 0.3) (type solid)) (layer "Dwgs.User"))
+    (fp_line (start 0.25 0) (end -0.75 1)
+      (stroke (width 0.3) (type solid)) (layer "Dwgs.User"))
+    (fp_line (start 0.25 1) (end 0.25 -1)
+      (stroke (width 0.3) (type solid)) (layer "Dwgs.User"))
+  )
   (footprint "LED_SMD:LED_WS2812B_PLCC4_5.0x5.0mm_P3.2mm" (layer "F.Cu")
     (at 150 63.7 180)
@@
     (pad "6" smd rect (at -5.9 0 180) (size 0.8 0.4) (layers "B.Cu" "B.Paste" "B.Mask")
       (net 21 "unconnected-(U2-GPIO3{slash}ADC1_CH3-Pad6)") (pinfunction "GPIO3/ADC1_CH3") (pintype "bidirectional"))
-    (pad "7" smd rect (at -5.9 -0.8 180) (size 0.8 0.4) (layers "B.Cu" "B.Paste" "B.Mask"))
+    (pad "7" smd rect (at -5.9 -0.8 180) (size 0.8 0.4) (layers "B.Cu" "B.Paste" "B.Mask")
+      (net 3 "+3.3V"))
     (pad "8" smd rect (at -5.9 -1.6 180) (size 0.8 0.4) (layers "B.Cu" "B.Paste" "B.Mask")
       (net 4 "/EN") (pinfunction "EN/CHIP_PU") (pintype "input"))
@@
   (gr_arc (start 156.025 125) (mid 155.732107 125.707107) (end 155.025 126)
     (stroke (width 0.1) (type solid)) (layer "Edge.Cuts"))
-  (gr_line (start 160.001855 98.033019) (end 160 114)
+  (gr_line (start 160.001855 98.033019) (end 160.001855 114)
     (stroke (width 0.1) (type solid)) (layer "Edge.Cuts"))
-  (gr_line (start 143.97 114) (end 140 114)
+  (gr_line (start 142.97 114) (end 140 114)
     (stroke (width 0.1) (type solid)) (layer "Edge.Cuts"))
   (gr_arc (start 144.975 126) (mid 144.267893 125.707107) (end 143.975 125)
     (stroke (width 0.1) (type solid)) (layer "Edge.Cuts"))
-  (gr_line (start 156.025 125) (end 156.03 114)
+  (gr_line (start 156.025 125) (end 156.027107 114.997107)
+    (stroke (width 0.1) (type solid)) (layer "Edge.Cuts"))
+  (gr_arc (start 142.97 114) (mid 143.677107 114.292893) (end 143.97 115)
+    (stroke (width 0.1) (type solid)) (layer "Edge.Cuts"))
+  (gr_line (start 143.97 115) (end 143.975 125)
     (stroke (width 0.1) (type solid)) (layer "Edge.Cuts"))
-  (gr_line (start 143.97 114) (end 143.975 125)
+  (gr_arc (start 156.027107 114.997107) (mid 156.32 114.29) (end 157.027107 113.997107)
     (stroke (width 0.1) (type solid)) (layer "Edge.Cuts"))
   (gr_arc (start 139.485643 97.16) (mid 139.861871 97.527029) (end 140 98.034157)
     (stroke (width 0.1) (type default)) (layer "Edge.Cuts"))
-  (gr_line (start 160 114) (end 156.03 114)
+  (gr_line (start 160.001855 114) (end 157.027107 113.997107)
     (stroke (width 0.1) (type solid)) (layer "Edge.Cuts"))
   (gr_arc (start 160.001855 98.033019) (mid 160.139984 97.525891) (end 160.516212 97.158862)
@@
   (via (at 145 116.3) (size 0.8) (drill 0.4) (layers "F.Cu" "B.Cu") (free) (net 2))
   (via (at 146 116.3) (size 0.8) (drill 0.4) (layers "F.Cu" "B.Cu") (free) (net 2))
+  (via (at 146.61 114.19) (size 0.8) (drill 0.4) (layers "F.Cu" "B.Cu") (free) (net 2))
   (via (at 154 108.91) (size 0.8) (drill 0.4) (layers "F.Cu" "B.Cu") (free) (net 2))
   (via (at 132.1 72.6) (size 0.8) (drill 0.4) (layers "F.Cu" "B.Cu") (free) (net 2))
   (via (at 151.4 125.4) (size 0.5) (drill 0.3) (layers "F.Cu" "B.Cu") (free) (net 2))
+  (via (at 147.6 114.2) (size 0.8) (drill 0.4) (layers "F.Cu" "B.Cu") (free) (net 2))
   (via (at 157.4 62.1) (size 0.8) (drill 0.4) (layers "F.Cu" "B.Cu") (free) (net 2))
   (via (at 150.99 101.5) (size 0.6) (drill 0.3) (layers "F.Cu" "B.Cu") (free) (net 2))
